Commit message: Adjusted the model parameters of gripper:   urdf/mikata_arm_4.urdf
Added model files of Mikata whose wrist is rotated:
  meshes/mikata_arm_4_joint5_rot.dae
  meshes/mikata_arm_4_joint5_rot.stl
  urdf/mikata_arm_4_rot.urdf

File: description/urdf/mikata_arm_4_rot.urdf (robot description, URDF)
Before this commit: robot mikata_arm_4, 8 links, 7 joints
Joints:
- joint gripper_joint_5: axis 0 0 -1 -> 0 -1 0; origin xyz=.04225 .015 0 rpy=0 0 0.2331650816 -> xyz=.04725 0 -.015 rpy=0 0.2331650816 0
- joint right_gripper_joint: axis 0 0 -1 -> 0 -1 0; origin xyz=.04225 -.015 0 rpy=0 0 -0.2331650816 -> xyz=.04725 0 .015 rpy=0 -0.2331650816 0
